Commit message: 整合piper_ros_moveit和piper_sim到piper_ros,修正urdf的质量和惯性矩阵,统一piper_description

File: src/piper_description/urdf/piper_description_gazebo.xacro (robot description, xacro)
@@ -23,19 +23,19 @@
       <geometry>
         <mesh
-          filename="package://piper_description/meshes/base_link.STL" />
-      </geometry>
-      <material
-        name="">
-        <color
-          rgba="0.792156862745098 0.819607843137255 0.933333333333333 1" />
-      </material>
-    </visual>
-    <collision>
-      <origin
-        xyz="0 0 0"
-        rpy="0 0 0" />
-      <geometry>
-        <mesh
-          filename="package://piper_description/meshes/base_link.STL" />
+          filename="file://$(find piper_description)/meshes/base_link.STL" />
+      </geometry>
+      <material
+        name="">
+        <color
+          rgba="0.792156862745098 0.819607843137255 0.933333333333333 1" />
+      </material>
+    </visual>
+    <collision>
+      <origin
+        xyz="0 0 0"
+        rpy="0 0 0" />
+      <geometry>
+        <mesh
+          filename="file://$(find piper_description)/meshes/base_link.STL" />
       </geometry>
     </collision>
@@ -54,19 +54,19 @@
       <geometry>
         <mesh
-          filename="package://piper_description/meshes/link1.STL" />
-      </geometry>
-      <material
-        name="">
-        <color
-          rgba="0.792156862745098 0.819607843137255 0.933333333333333 1" />
-      </material>
-    </visual>
-    <collision>
-      <origin
-        xyz="0 0 0"
-        rpy="0 0 0" />
-      <geometry>
-        <mesh
-          filename="package://piper_description/meshes/link1.STL" />
+          filename="file://$(find piper_description)/meshes/link1.STL" />
+      </geometry>
+      <material
+        name="">
+        <color
+          rgba="0.792156862745098 0.819607843137255 0.933333333333333 1" />
+      </material>
+    </visual>
+    <collision>
+      <origin
+        xyz="0 0 0"
+        rpy="0 0 0" />
+      <geometry>
+        <mesh
+          filename="file://$(find piper_description)/meshes/link1.STL" />
       </geometry>
     </collision>
@@ -103,19 +103,19 @@
       <geometry>
         <mesh
-          filename="package://piper_description/meshes/link2.STL" />
-      </geometry>
-      <material
-        name="">
-        <color
-          rgba="0.792156862745098 0.819607843137255 0.933333333333333 1" />
-      </material>
-    </visual>
-    <collision>
-      <origin
-        xyz="0 0 0"
-        rpy="0 0 0" />
-      <geometry>
-        <mesh
-          filename="package://piper_description/meshes/link2.STL" />
+          filename="file://$(find piper_description)/meshes/link2.STL" />
+      </geometry>
+      <material
+        name="">
+        <color
+          rgba="0.792156862745098 0.819607843137255 0.933333333333333 1" />
+      </material>
+    </visual>
+    <collision>
+      <origin
+        xyz="0 0 0"
+        rpy="0 0 0" />
+      <geometry>
+        <mesh
+          filename="file://$(find piper_description)/meshes/link2.STL" />
       </geometry>
     </collision>
@@ -152,19 +152,19 @@
       <geometry>
         <mesh
-          filename="package://piper_description/meshes/link3.STL" />
-      </geometry>
-      <material
-        name="">
-        <color
-          rgba="0.792156862745098 0.819607843137255 0.933333333333333 1" />
-      </material>
-    </visual>
-    <collision>
-      <origin
-        xyz="0 0 0"
-        rpy="0 0 0" />
-      <geometry>
-        <mesh
-          filename="package://piper_description/meshes/link3.STL" />
+          filename="file://$(find piper_description)/meshes/link3.STL" />
+      </geometry>
+      <material
+        name="">
+        <color
+          rgba="0.792156862745098 0.819607843137255 0.933333333333333 1" />
+      </material>
+    </visual>
+    <collision>
+      <origin
+        xyz="0 0 0"
+        rpy="0 0 0" />
+      <geometry>
+        <mesh
+          filename="file://$(find piper_description)/meshes/link3.STL" />
       </geometry>
     </collision>
@@ -201,19 +201,19 @@
       <geometry>
         <mesh
-          filename="package://piper_description/meshes/link4.STL" />
-      </geometry>
-      <material
-        name="">
-        <color
-          rgba="0.792156862745098 0.819607843137255 0.933333333333333 1" />
-      </material>
-    </visual>
-    <collision>
-      <origin
-        xyz="0 0 0"
-        rpy="0 0 0" />
-      <geometry>
-        <mesh
-          filename="package://piper_description/meshes/link4.STL" />
+          filename="file://$(find piper_description)/meshes/link4.STL" />
+      </geometry>
+      <material
+        name="">
+        <color
+          rgba="0.792156862745098 0.819607843137255 0.933333333333333 1" />
+      </material>
+    </visual>
+    <collision>
+      <origin
+        xyz="0 0 0"
+        rpy="0 0 0" />
+      <geometry>
+        <mesh
+          filename="file://$(find piper_description)/meshes/link4.STL" />
       </geometry>
     </collision>
@@ -250,19 +250,19 @@
       <geometry>
         <mesh
-          filename="package://piper_description/meshes/link5.STL" />
-      </geometry>
-      <material
-        name="">
-        <color
-          rgba="0.792156862745098 0.819607843137255 0.933333333333333 1" />
-      </material>
-    </visual>
-    <collision>
-      <origin
-        xyz="0 0 0"
-        rpy="0 0 0" />
-      <geometry>
-        <mesh
-          filename="package://piper_description/meshes/link5.STL" />
+          filename="file://$(find piper_description)/meshes/link5.STL" />
+      </geometry>
+      <material
+        name="">
+        <color
+          rgba="0.792156862745098 0.819607843137255 0.933333333333333 1" />
+      </material>
+    </visual>
+    <collision>
+      <origin
+        xyz="0 0 0"
+        rpy="0 0 0" />
+      <geometry>
+        <mesh
+          filename="file://$(find piper_description)/meshes/link5.STL" />
       </geometry>
     </collision>
@@ -299,5 +299,5 @@
       <geometry>
         <mesh
-          filename="package://piper_description/meshes/link6.STL" />
+          filename="file://$(find piper_description)/meshes/link6.STL" />
       </geometry>
       <material
@@ -313,5 +313,5 @@
       <geometry>
         <mesh
-          filename="package://piper_description/meshes/link6.STL" />
+          filename="file://$(find piper_description)/meshes/link6.STL" />
       </geometry>
     </collision>
@@ -357,19 +357,19 @@
       <geometry>
         <mesh
-          filename="package://piper_description/meshes/gripper_base.STL" />
-      </geometry>
-      <material
-        name="">
-        <color
-          rgba="0.792156862745098 0.819607843137255 0.933333333333333 1" />
-      </material>
-    </visual>
-    <collision>
-      <origin
-        xyz="0 0 0"
-        rpy="0 0 0" />
-      <geometry>
-        <mesh
-          filename="package://piper_description/meshes/gripper_base.STL" />
+          filename="file://$(find piper_description)/meshes/gripper_base.STL" />
+      </geometry>
+      <material
+        name="">
+        <color
+          rgba="0.792156862745098 0.819607843137255 0.933333333333333 1" />
+      </material>
+    </visual>
+    <collision>
+      <origin
+        xyz="0 0 0"
+        rpy="0 0 0" />
+      <geometry>
+        <mesh
+          filename="file://$(find piper_description)/meshes/gripper_base.STL" />
       </geometry>
     </collision>
@@ -408,19 +408,19 @@
       <geometry>
         <mesh
-          filename="package://piper_description/meshes/link7.STL" />
-      </geometry>
-      <material
-        name="">
-        <color
-          rgba="0.792156862745098 0.819607843137255 0.933333333333333 1" />
-      </material>
-    </visual>
-    <collision>
-      <origin
-        xyz="0 0 0"
-        rpy="0 0 0" />
-      <geometry>
-        <mesh
-          filename="package://piper_description/meshes/link7.STL" />
+          filename="file://$(find piper_description)/meshes/link7.STL" />
+      </geometry>
+      <material
+        name="">
+        <color
+          rgba="0.792156862745098 0.819607843137255 0.933333333333333 1" />
+      </material>
+    </visual>
+    <collision>
+      <origin
+        xyz="0 0 0"
+        rpy="0 0 0" />
+      <geometry>
+        <mesh
+          filename="file://$(find piper_description)/meshes/link7.STL" />
       </geometry>
     </collision>
@@ -466,19 +466,19 @@
       <geometry>
         <mesh
-          filename="package://piper_description/meshes/link8.STL" />
-      </geometry>
-      <material
-        name="">
-        <color
-          rgba="0.792156862745098 0.819607843137255 0.933333333333333 1" />
-      </material>
-    </visual>
-    <collision>
-      <origin
-        xyz="0 0 0"
-        rpy="0 0 0" />
-      <geometry>
-        <mesh
-          filename="package://piper_description/meshes/link8.STL" />
+          filename="file://$(find piper_description)/meshes/link8.STL" />
+      </geometry>
+      <material
+        name="">
+        <color
+          rgba="0.792156862745098 0.819607843137255 0.933333333333333 1" />
+      </material>
+    </visual>
+    <collision>
+      <origin
+        xyz="0 0 0"
+        rpy="0 0 0" />
+      <geometry>
+        <mesh
+          filename="file://$(find piper_description)/meshes/link8.STL" />
       </geometry>
     </collision>
@@ -502,59 +502,126 @@
       velocity="1" />
   </joint>
-<!-- controller -->
-  <xacro:macro name="transmission_block" params="tran_name joint_name motor_name">
-    <transmission name="${tran_name}">
-        <type>transmission_interface/SimpleTransmission</type>
-        <joint name="${joint_name}">
-            <hardwareInterface>hardware_interface/PositionJointInterface</hardwareInterface>
-        </joint>
-        <actuator name="$motor_name">
-            <hardwareInterface>hardware_interface/PositionJointInterface</hardwareInterface>
-            <mechanicalReduction>1</mechanicalReduction>
-        </actuator>
-    </transmission>
-  </xacro:macro>
-  <xacro:transmission_block tran_name="tran1" joint_name="joint1" motor_name="motor1"/>
-  <xacro:transmission_block tran_name="tran2" joint_name="joint2" motor_name="motor2"/>
-  <xacro:transmission_block tran_name="tran3" joint_name="joint3" motor_name="motor3"/>
-  <xacro:transmission_block tran_name="tran4" joint_name="joint4" motor_name="motor4"/>
-  <xacro:transmission_block tran_name="tran5" joint_name="joint5" motor_name="motor5"/>
-  <xacro:transmission_block tran_name="tran6" joint_name="joint6" motor_name="motor6"/>
-  <xacro:transmission_block tran_name="tran7" joint_name="joint7" motor_name="motor7"/>
-  <xacro:transmission_block tran_name="tran8" joint_name="joint8" motor_name="motor8"/>
+  <!-- <gazebo reference="base_link">
+      <material>Gazebo/Black</material>
+      <gravity>true</gravity>
+      <selfCollide>false</selfCollide>
+  </gazebo>
+  <gazebo reference="link1">
+      <material>Gazebo/Gray</material>
+      <selfCollide>false</selfCollide>
+  </gazebo>
+  <gazebo reference="link2">
+      <material>Gazebo/Red</material>
+      <selfCollide>false</selfCollide>
+  </gazebo>
+  <gazebo reference="link3">
+      <material>Gazebo/Blue</material>
+  </gazebo>
+  <gazebo reference="link4">
+      <material>Gazebo/Green</material>
+  </gazebo>
+  <gazebo reference="link5">
+      <material>Gazebo/Yellow</material>
+  </gazebo>
+  <gazebo reference="link6">
+      <material>Gazebo/Orange</material>
+  </gazebo>
+  <gazebo reference="link7">
+      <material>Gazebo/Orange</material>
+  </gazebo>
+  <gazebo reference="link8">
+      <material>Gazebo/Orange</material>
+  </gazebo> -->
+  <ros2_control name="GazeboSystem" type="system">
+      <hardware>
+          <plugin>gazebo_ros2_control/GazeboSystem</plugin>
+      </hardware>
+      <joint name="joint1">
+          <command_interface name="position">
+              <param name="min">-1</param>
+              <param name="max">1</param>
+          </command_interface>
+          <state_interface name="position">
+              <param name="initial_value">0.0</param>
+          </state_interface>
+          <state_interface name="velocity"/>
+      </joint>
+      <joint name="joint2">
+          <command_interface name="position">
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
File: src/piper_description/urdf/piper_no_gripper_description.xacro (robot description, xacro)
@@ -356,6 +356,6 @@
 <!-- gazebo -->
   <gazebo>
-    <plugin name="gazebo_ros_control" filename="libgazebo_ros_control.so">
-        <robotNamespace>/piper_description</robotNamespace>
+    <plugin name="gazebo_ros2_control" filename="libgazebo_ros2_control.so">
+        <robotNamespace>/piper</robotNamespace>
         <legacyModeNS>true</legacyModeNS>
     </plugin>
