Commit message: 整合piper_ros_moveit和piper_sim到piper_ros,修正urdf的质量和惯性矩阵,统一piper_description

File: src/piper_description/urdf/piper_no_gripper_description_gazebo.xacro (robot description, xacro)
@@ -23,19 +23,19 @@
       <geometry>
         <mesh
-          filename="package://piper_description/meshes/base_link.STL" />
-      </geometry>
-      <material
-        name="">
-        <color
-          rgba="0.792156862745098 0.819607843137255 0.933333333333333 1" />
-      </material>
-    </visual>
-    <collision>
-      <origin
-        xyz="0 0 0"
-        rpy="0 0 0" />
-      <geometry>
-        <mesh
-          filename="package://piper_description/meshes/base_link.STL" />
+          filename="file://$(find piper_description)/meshes/base_link.STL" />
+      </geometry>
+      <material
+        name="">
+        <color
+          rgba="0.792156862745098 0.819607843137255 0.933333333333333 1" />
+      </material>
+    </visual>
+    <collision>
+      <origin
+        xyz="0 0 0"
+        rpy="0 0 0" />
+      <geometry>
+        <mesh
+          filename="file://$(find piper_description)/meshes/base_link.STL" />
       </geometry>
     </collision>
@@ -54,19 +54,19 @@
       <geometry>
         <mesh
-          filename="package://piper_description/meshes/link1.STL" />
-      </geometry>
-      <material
-        name="">
-        <color
-          rgba="0.792156862745098 0.819607843137255 0.933333333333333 1" />
-      </material>
-    </visual>
-    <collision>
-      <origin
-        xyz="0 0 0"
-        rpy="0 0 0" />
-      <geometry>
-        <mesh
-          filename="package://piper_description/meshes/link1.STL" />
+          filename="file://$(find piper_description)/meshes/link1.STL" />
+      </geometry>
+      <material
+        name="">
+        <color
+          rgba="0.792156862745098 0.819607843137255 0.933333333333333 1" />
+      </material>
+    </visual>
+    <collision>
+      <origin
+        xyz="0 0 0"
+        rpy="0 0 0" />
+      <geometry>
+        <mesh
+          filename="file://$(find piper_description)/meshes/link1.STL" />
       </geometry>
     </collision>
@@ -103,19 +103,19 @@
       <geometry>
         <mesh
-          filename="package://piper_description/meshes/link2.STL" />
-      </geometry>
-      <material
-        name="">
-        <color
-          rgba="0.792156862745098 0.819607843137255 0.933333333333333 1" />
-      </material>
-    </visual>
-    <collision>
-      <origin
-        xyz="0 0 0"
-        rpy="0 0 0" />
-      <geometry>
-        <mesh
-          filename="package://piper_description/meshes/link2.STL" />
+          filename="file://$(find piper_description)/meshes/link2.STL" />
+      </geometry>
+      <material
+        name="">
+        <color
+          rgba="0.792156862745098 0.819607843137255 0.933333333333333 1" />
+      </material>
+    </visual>
+    <collision>
+      <origin
+        xyz="0 0 0"
+        rpy="0 0 0" />
+      <geometry>
+        <mesh
+          filename="file://$(find piper_description)/meshes/link2.STL" />
       </geometry>
     </collision>
@@ -152,19 +152,19 @@
       <geometry>
         <mesh
-          filename="package://piper_description/meshes/link3.STL" />
-      </geometry>
-      <material
-        name="">
-        <color
-          rgba="0.792156862745098 0.819607843137255 0.933333333333333 1" />
-      </material>
-    </visual>
-    <collision>
-      <origin
-        xyz="0 0 0"
-        rpy="0 0 0" />
-      <geometry>
-        <mesh
-          filename="package://piper_description/meshes/link3.STL" />
+          filename="file://$(find piper_description)/meshes/link3.STL" />
+      </geometry>
+      <material
+        name="">
+        <color
+          rgba="0.792156862745098 0.819607843137255 0.933333333333333 1" />
+      </material>
+    </visual>
+    <collision>
+      <origin
+        xyz="0 0 0"
+        rpy="0 0 0" />
+      <geometry>
+        <mesh
+          filename="file://$(find piper_description)/meshes/link3.STL" />
       </geometry>
     </collision>
@@ -201,19 +201,19 @@
       <geometry>
         <mesh
-          filename="package://piper_description/meshes/link4.STL" />
-      </geometry>
-      <material
-        name="">
-        <color
-          rgba="0.792156862745098 0.819607843137255 0.933333333333333 1" />
-      </material>
-    </visual>
-    <collision>
-      <origin
-        xyz="0 0 0"
-        rpy="0 0 0" />
-      <geometry>
-        <mesh
-          filename="package://piper_description/meshes/link4.STL" />
+          filename="file://$(find piper_description)/meshes/link4.STL" />
+      </geometry>
+      <material
+        name="">
+        <color
+          rgba="0.792156862745098 0.819607843137255 0.933333333333333 1" />
+      </material>
+    </visual>
+    <collision>
+      <origin
+        xyz="0 0 0"
+        rpy="0 0 0" />
+      <geometry>
+        <mesh
+          filename="file://$(find piper_description)/meshes/link4.STL" />
       </geometry>
     </collision>
@@ -250,19 +250,19 @@
       <geometry>
         <mesh
-          filename="package://piper_description/meshes/link5.STL" />
-      </geometry>
-      <material
-        name="">
-        <color
-          rgba="0.792156862745098 0.819607843137255 0.933333333333333 1" />
-      </material>
-    </visual>
-    <collision>
-      <origin
-        xyz="0 0 0"
-        rpy="0 0 0" />
-      <geometry>
-        <mesh
-          filename="package://piper_description/meshes/link5.STL" />
+          filename="file://$(find piper_description)/meshes/link5.STL" />
+      </geometry>
+      <material
+        name="">
+        <color
+          rgba="0.792156862745098 0.819607843137255 0.933333333333333 1" />
+      </material>
+    </visual>
+    <collision>
+      <origin
+        xyz="0 0 0"
+        rpy="0 0 0" />
+      <geometry>
+        <mesh
+          filename="file://$(find piper_description)/meshes/link5.STL" />
       </geometry>
     </collision>
@@ -299,5 +299,5 @@
       <geometry>
         <mesh
-          filename="package://piper_description/meshes/link6.STL" />
+          filename="file://$(find piper_description)/meshes/link6.STL" />
       </geometry>
       <material
@@ -313,5 +313,5 @@
       <geometry>
         <mesh
-          filename="package://piper_description/meshes/link6.STL" />
+          filename="file://$(find piper_description)/meshes/link6.STL" />
       </geometry>
     </collision>
@@ -335,226 +335,100 @@
       velocity="3" />
   </joint>
-  <link
-    name="gripper_base">
-    <inertial>
-      <origin
-        xyz="-0.000183807162235591 8.05033155577911E-05 0.0321436689908876"
-        rpy="0 0 0" />
-      <mass
-        value="0.45" />
-      <inertia
-        ixx="0.00092934"
-        ixy="0.00000034"
-        ixz="-0.00000738"
-        iyy="0.00071447"
-        iyz="0.00000005"
-        izz="0.00039442" />
-    </inertial>
-    <visual>
-      <origin
-        xyz="0 0 0"
-        rpy="0 0 0" />
-      <geometry>
-        <mesh
-          filename="package://piper_description/meshes/gripper_base.STL" />
-      </geometry>
-      <material
-        name="">
-        <color
-          rgba="0.792156862745098 0.819607843137255 0.933333333333333 1" />
-      </material>
-    </visual>
-    <collision>
-      <origin
-        xyz="0 0 0"
-        rpy="0 0 0" />
-      <geometry>
-        <mesh
-          filename="package://piper_description/meshes/gripper_base.STL" />
-      </geometry>
-    </collision>
-  </link>
-  <joint
-    name="joint6_to_gripper_base"
-    type="fixed">
-    <origin
-      xyz="0 0 0"
-      rpy="0 0 0" />
-    <parent
-      link="link6" />
-    <child
-      link="gripper_base" />
-  </joint>
-  <link
-    name="link7">
-    <inertial>
-      <origin
-        xyz="0.00065123185041968 -0.0491929869131989 0.00972258769184025"
-        rpy="0 0 0" />
-      <mass
-        value="0.025" />
-      <inertia
-        ixx="0.00007371"
-        ixy="-0.00000113"
-        ixz="0.00000021"
-        iyy="-0.00000113"
-        iyz="-0.00001372"
-        izz="0.0000747" />
-    </inertial>
-    <visual>
-      <origin
-        xyz="0 0 0"
-        rpy="0 0 0" />
-      <geometry>
-        <mesh
-          filename="package://piper_description/meshes/link7.STL" />
-      </geometry>
-      <material
-        name="">
-        <color
-          rgba="0.792156862745098 0.819607843137255 0.933333333333333 1" />
-      </material>
-    </visual>
-    <collision>
-      <origin
-        xyz="0 0 0"
-        rpy="0 0 0" />
-      <geometry>
-        <mesh
-          filename="package://piper_description/meshes/link7.STL" />
-      </geometry>
-    </collision>
-  </link>
-  <joint
-    name="joint7"
-    type="prismatic">
-    <origin
-      xyz="0 0 0.1358"
-      rpy="1.5708 0 0" />
-    <parent
-      link="gripper_base" />
-    <child
-      link="link7" />
-    <axis
-      xyz="0 0 1" />
-    <limit
-      lower="0"
-      upper="0.035"
-      effort="10"
-      velocity="1" />
-  </joint>
-  <link
-    name="link8">
-    <inertial>
-      <origin
-        xyz="0.000651231850419722 -0.0491929869131991 0.00972258769184024"
-        rpy="0 0 0" />
-      <mass
-        value="0.025" />
-      <inertia
-        ixx="0.00007371"
-        ixy="-0.00000113"
-        ixz="0.00000021"
-        iyy="-0.00000113"
-        iyz="-0.00001372"
-        izz="0.0000747" />
-    </inertial>
-    <visual>
-      <origin
-        xyz="0 0 0"
-        rpy="0 0 0" />
-      <geometry>
-        <mesh
-          filename="package://piper_description/meshes/link8.STL" />
-      </geometry>
-      <material
-        name="">
-        <color
-          rgba="0.792156862745098 0.819607843137255 0.933333333333333 1" />
-      </material>
-    </visual>
-    <collision>
-      <origin
-        xyz="0 0 0"
-        rpy="0 0 0" />
-      <geometry>
-        <mesh
-          filename="package://piper_description/meshes/link8.STL" />
-      </geometry>
-    </collision>
-  </link>
-  <joint
-    name="joint8"
-    type="prismatic">
-    <origin
-      xyz="0 0 0.1358"
-      rpy="1.5708 0 -3.1416" />
-    <parent
-      link="gripper_base" />
-    <child
-      link="link8" />
-    <axis
-      xyz="0 0 -1" />
-    <limit
-      lower="-0.035"
-      upper="0"
-      effort="10"
-      velocity="1" />
-  </joint>
-<!-- controller -->
-  <xacro:macro name="transmission_block" params="tran_name joint_name motor_name">
-    <transmission name="${tran_name}">
-        <type>transmission_interface/SimpleTransmission</type>
-        <joint name="${joint_name}">
-            <hardwareInterface>hardware_interface/PositionJointInterface</hardwareInterface>
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